File: Kicad/rj45-tester-receiver/rj45-tester-receiver.sch (KiCad schematic (older format))
At the start: 17 parts

Commit message: PCB receiver
Parts:
- D1, D11, D13, D15, D3, D5, D7, D9: renamed from D?; footprint (none) -> LED_SMD:LED_0805_2012Metric_Pad1.15x1.40mm_HandSolder
- D10, D12, D14, D16, D2, D4, D6, D8: renamed from D?; footprint (none) -> Diode_SMD:D_0805_2012Metric_Pad1.15x1.40mm_HandSolder
- J1: renamed from J?; footprint (none) -> Connector_RJ:RJ45_Amphenol_54602-x08_Horizontal
Changed lines of the file:
@@
 $EndDescr
 $Comp
-L Connector:RJ45 J?
+L Connector:RJ45 J1
 U 1 1 5F5D1739
 P 3650 3600
-F 0 "J?" H 3707 4267 50  0000 C CNN
+F 0 "J1" H 3707 4267 50  0000 C CNN
 F 1 "RJ45" H 3707 4176 50  0000 C CNN
-F 2 "" V 3650 3625 50  0001 C CNN
+F 2 "Connector_RJ:RJ45_Amphenol_54602-x08_Horizontal" V 3650 3625 50  0001 C CNN
 F 3 "~" V 3650 3625 50  0001 C CNN
 	1    3650 3600
@@
 $EndComp
 $Comp
-L Device:LED D?
+L Device:LED D3
 U 1 1 5F5D1E03
 P 5650 2350
-F 0 "D?" H 5600 2250 50  0000 C CNN
+F 0 "D3" H 5600 2250 50  0000 C CNN
 F 1 "LED" H 5750 2250 50  0000 C CNN
-F 2 "" H 5650 2350 50  0001 C CNN
+F 2 "LED_SMD:LED_0805_2012Metric_Pad1.15x1.40mm_HandSolder" H 5650 2350 50  0001 C CNN
 F 3 "~" H 5650 2350 50  0001 C CNN
 	1    5650 2350
@@
 $EndComp
 $Comp
-L Device:D D?
+L Device:D D4
 U 1 1 5F5D230C
 P 5650 2600
-F 0 "D?" H 5700 2700 50  0000 C CNN
+F 0 "D4" H 5700 2700 50  0000 C CNN
 F 1 "D" H 5600 2700 50  0000 C CNN
-F 2 "" H 5650 2600 50  0001 C CNN
+F 2 "Diode_SMD:D_0805_2012Metric_Pad1.15x1.40mm_HandSolder" H 5650 2600 50  0001 C CNN
 F 3 "~" H 5650 2600 50  0001 C CNN
 	1    5650 2600
@@
 	5900 2600 5800 2600
 $Comp
-L Device:LED D?
+L Device:LED D5
 U 1 1 5F5D4785
 P 5650 2850
-F 0 "D?" H 5600 2750 50  0000 C CNN
+F 0 "D5" H 5600 2750 50  0000 C CNN
 F 1 "LED" H 5750 2750 50  0000 C CNN
-F 2 "" H 5650 2850 50  0001 C CNN
+F 2 "LED_SMD:LED_0805_2012Metric_Pad1.15x1.40mm_HandSolder" H 5650 2850 50  0001 C CNN
 F 3 "~" H 5650 2850 50  0001 C CNN
 	1    5650 2850
@@
 $EndComp
 $Comp
-L Device:D D?
+L Device:D D6
 U 1 1 5F5D478B
 P 5650 3100
-F 0 "D?" H 5700 3200 50  0000 C CNN
+F 0 "D6" H 5700 3200 50  0000 C CNN
 F 1 "D" H 5600 3200 50  0000 C CNN
-F 2 "" H 5650 3100 50  0001 C CNN
+F 2 "Diode_SMD:D_0805_2012Metric_Pad1.15x1.40mm_HandSolder" H 5650 3100 50  0001 C CNN
 F 3 "~" H 5650 3100 50  0001 C CNN
 	1    5650 3100
@@
 	5900 3100 5800 3100
 $Comp
-L Device:LED D?
+L Device:LED D7
 U 1 1 5F5D51BB
 P 5650 3350
-F 0 "D?" H 5600 3250 50  0000 C CNN
+F 0 "D7" H 5600 3250 50  0000 C CNN
 F 1 "LED" H 5750 3250 50  0000 C CNN
-F 2 "" H 5650 3350 50  0001 C CNN
+F 2 "LED_SMD:LED_0805_2012Metric_Pad1.15x1.40mm_HandSolder" H 5650 3350 50  0001 C CNN
 F 3 "~" H 5650 3350 50  0001 C CNN
 	1    5650 3350
@@
 $EndComp
 $Comp
-L Device:D D?
+L Device:D D8
 U 1 1 5F5D51C1
 P 5650 3600
-F 0 "D?" H 5700 3700 50  0000 C CNN
+F 0 "D8" H 5700 3700 50  0000 C CNN
 F 1 "D" H 5600 3700 50  0000 C CNN
-F 2 "" H 5650 3600 50  0001 C CNN
+F 2 "Diode_SMD:D_0805_2012Metric_Pad1.15x1.40mm_HandSolder" H 5650 3600 50  0001 C CNN
 F 3 "~" H 5650 3600 50  0001 C CNN
 	1    5650 3600
@@
 	5900 3600 5800 3600
 $Comp
-L Device:LED D?
+L Device:LED D9
 U 1 1 5F5D5C21
 P 5650 3850
-F 0 "D?" H 5600 3750 50  0000 C CNN
+F 0 "D9" H 5600 3750 50  0000 C CNN
 F 1 "LED" H 5750 3750 50  0000 C CNN
-F 2 "" H 5650 3850 50  0001 C CNN
+F 2 "LED_SMD:LED_0805_2012Metric_Pad1.15x1.40mm_HandSolder" H 5650 3850 50  0001 C CNN
 F 3 "~" H 5650 3850 50  0001 C CNN
 	1    5650 3850
@@
 $EndComp
 $Comp
-L Device:D D?
+L Device:D D10
 U 1 1 5F5D5C27
 P 5650 4100
-F 0 "D?" H 5700 4200 50  0000 C CNN
+F 0 "D10" H 5700 4200 50  0000 C CNN
 F 1 "D" H 5600 4200 50  0000 C CNN
-F 2 "" H 5650 4100 50  0001 C CNN
+F 2 "Diode_SMD:D_0805_2012Metric_Pad1.15x1.40mm_HandSolder" H 5650 4100 50  0001 C CNN
 F 3 "~" H 5650 4100 50  0001 C CNN
 	1    5650 4100
@@
 	5900 4100 5800 4100
 $Comp
-L Device:LED D?
+L Device:LED D11
 U 1 1 5F5D5F11
 P 5650 4350
-F 0 "D?" H 5600 4250 50  0000 C CNN
+F 0 "D11" H 5600 4250 50  0000 C CNN
 F 1 "LED" H 5750 4250 50  0000 C CNN
-F 2 "" H 5650 4350 50  0001 C CNN
+F 2 "LED_SMD:LED_0805_2012Metric_Pad1.15x1.40mm_HandSolder" H 5650 4350 50  0001 C CNN
 F 3 "~" H 5650 4350 50  0001 C CNN
 	1    5650 4350
@@
 $EndComp
 $Comp
-L Device:D D?
+L Device:D D12
 U 1 1 5F5D5F17
 P 5650 4600
-F 0 "D?" H 5700 4700 50  0000 C CNN
+F 0 "D12" H 5700 4700 50  0000 C CNN
 F 1 "D" H 5600 4700 50  0000 C CNN
-F 2 "" H 5650 4600 50  0001 C CNN
+F 2 "Diode_SMD:D_0805_2012Metric_Pad1.15x1.40mm_HandSolder" H 5650 4600 50  0001 C CNN
 F 3 "~" H 5650 4600 50  0001 C CNN
 	1    5650 4600
@@
 	5900 4600 5800 4600
 $Comp
-L Device:LED D?
+L Device:LED D13
 U 1 1 5F5D653C
 P 5650 4850
-F 0 "D?" H 5600 4750 50  0000 C CNN
+F 0 "D13" H 5600 4750 50  0000 C CNN
 F 1 "LED" H 5750 4750 50  0000 C CNN
-F 2 "" H 5650 4850 50  0001 C CNN
+F 2 "LED_SMD:LED_0805_2012Metric_Pad1.15x1.40mm_HandSolder" H 5650 4850 50  0001 C CNN
 F 3 "~" H 5650 4850 50  0001 C CNN
 	1    5650 4850
@@
 $EndComp
 $Comp
-L Device:D D?
+L Device:D D14
 U 1 1 5F5D6542
 P 5650 5100
-F 0 "D?" H 5700 5200 50  0000 C CNN
+F 0 "D14" H 5700 5200 50  0000 C CNN
 F 1 "D" H 5600 5200 50  0000 C CNN
-F 2 "" H 5650 5100 50  0001 C CNN
+F 2 "Diode_SMD:D_0805_2012Metric_Pad1.15x1.40mm_HandSolder" H 5650 5100 50  0001 C CNN
 F 3 "~" H 5650 5100 50  0001 C CNN
 	1    5650 5100
@@
 	5800 5350 5900 5350
 $Comp
-L Device:D D?
+L Device:D D16
 U 1 1 5F5D6A23
 P 5650 5600
-F 0 "D?" H 5700 5700 50  0000 C CNN
+F 0 "D16" H 5700 5700 50  0000 C CNN
 F 1 "D" H 5600 5700 50  0000 C CNN
-F 2 "" H 5650 5600 50  0001 C CNN
+F 2 "Diode_SMD:D_0805_2012Metric_Pad1.15x1.40mm_HandSolder" H 5650 5600 50  0001 C CNN
 F 3 "~" H 5650 5600 50  0001 C CNN
 	1    5650 5600
@@
 $EndComp
 $Comp
-L Device:LED D?
+L Device:LED D15
 U 1 1 5F5D6A1D
 P 5650 5350
-F 0 "D?" H 5600 5250 50  0000 C CNN
+F 0 "D15" H 5600 5250 50  0000 C CNN
 F 1 "LED" H 5750 5250 50  0000 C CNN
-F 2 "" H 5650 5350 50  0001 C CNN
+F 2 "LED_SMD:LED_0805_2012Metric_Pad1.15x1.40mm_HandSolder" H 5650 5350 50  0001 C CNN
 F 3 "~" H 5650 5350 50  0001 C CNN
 	1    5650 5350
@@
 	5350 2350 5350 2450
 $Comp
-L Device:LED D?
+L Device:LED D1
 U 1 1 5F5F8D46
 P 5650 1850
-F 0 "D?" H 5600 1750 50  0000 C CNN
+F 0 "D1" H 5600 1750 50  0000 C CNN
 F 1 "LED" H 5750 1750 50  0000 C CNN
-F 2 "" H 5650 1850 50  0001 C CNN
+F 2 "LED_SMD:LED_0805_2012Metric_Pad1.15x1.40mm_HandSolder" H 5650 1850 50  0001 C CNN
 F 3 "~" H 5650 1850 50  0001 C CNN
 	1    5650 1850
@@
 $EndComp
 $Comp
-L Device:D D?
+L Device:D D2
 U 1 1 5F5F8D4C
 P 5650 2100
-F 0 "D?" H 5700 2200 50  0000 C CNN
+F 0 "D2" H 5700 2200 50  0000 C CNN
 F 1 "D" H 5600 2200 50  0000 C CNN
-F 2 "" H 5650 2100 50  0001 C CNN
+F 2 "Diode_SMD:D_0805_2012Metric_Pad1.15x1.40mm_HandSolder" H 5650 2100 50  0001 C CNN
 F 3 "~" H 5650 2100 50  0001 C CNN
 	1    5650 2100
