File: Kicad/rj45-tester-emitter/rj45-tester-emitter.kicad_pcb (KiCad board)
At the start: 2 copper layers, 40 x 60 mm, 30 parts, among them J1 Conn_01x02_Male, J2 RJ45, SW1 SW_Push_SPDT, U1 NE555P, U2 4017

Commit message: PCB receiver
Routing:
- net Net-(D4-Pad2): track 35.3 -> 33.2 mm

Commit message: Drill Holes
Parts:
- added REF**: MountingHole_3mm, MountingHole:MountingHole_3mm, F.Cu at (103.4, 106.6)
- added REF**: MountingHole_3mm, MountingHole:MountingHole_3mm, F.Cu at (136.6, 106.6)
- added REF**: MountingHole_3mm, MountingHole:MountingHole_3mm, F.Cu at (136.6, 53.4)
- added REF**: MountingHole_3mm, MountingHole:MountingHole_3mm, F.Cu at (103.4, 53.4)
Other:
- outline, holes or cut-outs redrawn
Changed lines of the file:
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@@
   (general
     (thickness 1.6)
-    (drawings 20)
+    (drawings 16)
     (tracks 175)
     (zones 0)
-    (modules 30)
+    (modules 34)
     (nets 29)
   )
@@
     (38 B.Mask user hide)
     (39 F.Mask user hide)
-    (40 Dwgs.User user hide)
+    (40 Dwgs.User user)
     (41 Cmts.User user hide)
     (42 Eco1.User user)
@@
     (visible_elements 7FFBFFFF)
     (pcbplotparams
-      (layerselection 0x010fc_ffffffff)
+      (layerselection 0x010f0_ffffffff)
       (usegerberextensions false)
       (usegerberattributes true)
@@
       (outputformat 1)
       (mirror false)
-      (drillshape 1)
+      (drillshape 0)
       (scaleselection 1)
       (outputdirectory ""))
@@
     (add_net "Net-(J1-Pad1)")
     (add_net VCC)
+  )
+  (module MountingHole:MountingHole_3mm (layer F.Cu)
+    (at 103.4 106.6)
+    (descr "Mounting Hole 3mm, no annular")
+    (tags "mounting hole 3mm no annular")
+    (attr virtual)
+    (fp_text reference REF** (at 0 -4) (layer F.SilkS) hide
+      (effects (font (size 1 1) (thickness 0.15)))
+    )
+    (fp_text value MountingHole_3mm (at 0 4) (layer F.Fab)
+      (effects (font (size 1 1) (thickness 0.15)))
+    )
+    (fp_text user %R (at 0.3 0) (layer F.Fab)
+      (effects (font (size 1 1) (thickness 0.15)))
+    )
+    (fp_circle (center 0 0) (end 3 0) (layer Cmts.User) (width 0.15))
+    (fp_circle (center 0 0) (end 3.25 0) (layer F.CrtYd) (width 0.05))
+    (pad 1 np_thru_hole circle (at 0 0) (size 3 3) (drill 3) (layers *.Cu *.Mask))
+  )
+  (module MountingHole:MountingHole_3mm (layer F.Cu)
+    (at 136.6 106.6)
+    (descr "Mounting Hole 3mm, no annular")
+    (tags "mounting hole 3mm no annular")
+    (attr virtual)
+    (fp_text reference REF** (at 0 -4) (layer F.SilkS) hide
+      (effects (font (size 1 1) (thickness 0.15)))
+    )
+    (fp_text value MountingHole_3mm (at 0 4) (layer F.Fab)
+      (effects (font (size 1 1) (thickness 0.15)))
+    )
+    (fp_text user %R (at 0.3 0) (layer F.Fab)
+      (effects (font (size 1 1) (thickness 0.15)))
+    )
+    (fp_circle (center 0 0) (end 3 0) (layer Cmts.User) (width 0.15))
+    (fp_circle (center 0 0) (end 3.25 0) (layer F.CrtYd) (width 0.05))
+    (pad 1 np_thru_hole circle (at 0 0) (size 3 3) (drill 3) (layers *.Cu *.Mask))
+  )
+  (module MountingHole:MountingHole_3mm (layer F.Cu)
+    (at 136.6 53.4)
+    (descr "Mounting Hole 3mm, no annular")
+    (tags "mounting hole 3mm no annular")
+    (attr virtual)
+    (fp_text reference REF** (at 0 -4) (layer F.SilkS) hide
+      (effects (font (size 1 1) (thickness 0.15)))
+    )
+    (fp_text value MountingHole_3mm (at 0 4) (layer F.Fab)
+      (effects (font (size 1 1) (thickness 0.15)))
+    )
+    (fp_text user %R (at 0.3 0) (layer F.Fab)
+      (effects (font (size 1 1) (thickness 0.15)))
+    )
+    (fp_circle (center 0 0) (end 3 0) (layer Cmts.User) (width 0.15))
+    (fp_circle (center 0 0) (end 3.25 0) (layer F.CrtYd) (width 0.05))
+    (pad 1 np_thru_hole circle (at 0 0) (size 3 3) (drill 3) (layers *.Cu *.Mask))
+  )
+  (module MountingHole:MountingHole_3mm (layer F.Cu)
+    (at 103.4 53.4)
+    (descr "Mounting Hole 3mm, no annular")
+    (tags "mounting hole 3mm no annular")
+    (attr virtual)
+    (fp_text reference REF** (at 0 -4) (layer F.SilkS) hide
+      (effects (font (size 1 1) (thickness 0.15)))
+    )
+    (fp_text value MountingHole_3mm (at 0 4) (layer F.Fab)
+      (effects (font (size 1 1) (thickness 0.15)))
+    )
+    (fp_text user %R (at 0.3 0) (layer F.Fab)
+      (effects (font (size 1 1) (thickness 0.15)))
+    )
+    (fp_circle (center 0 0) (end 3 0) (layer Cmts.User) (width 0.15))
+    (fp_circle (center 0 0) (end 3.25 0) (layer F.CrtYd) (width 0.05))
+    (pad 1 np_thru_hole circle (at 0 0) (size 3 3) (drill 3) (layers *.Cu *.Mask))
   )
   (module Symbol:OSHW-Symbol_6.7x6mm_SilkScreen (layer B.Cu)
@@
     (effects (font (size 1 1) (thickness 0.15)))
   )
-  (gr_circle (center 137 107) (end 139 107) (layer Edge.Cuts) (width 0.05))
-  (gr_circle (center 103 107) (end 105 107) (layer Edge.Cuts) (width 0.05))
-  (gr_circle (center 103 53) (end 105 53) (layer Edge.Cuts) (width 0.05))
-  (gr_circle (center 137 53) (end 139 53) (layer Edge.Cuts) (width 0.05))
   (dimension 40 (width 0.15) (layer Eco1.User)
     (gr_text "40.000 mm" (at 120 117.3) (layer Eco1.User)
